File: orienteringsklokke v3.sch (EAGLE design)
At the start: 16 parts

Commit message: Lots of work on version 3
Parts:
- removed S1: (no value), switch-omron:10-XX
- added LED2: (no value), led:LED3MM
- added R4: 220, resistor:R-EU_0204/5
- added U$5: PUSHBUTTON_2P, joakim:PUSHBUTTON_2P
- C1: device resistor:CPOL-EUE2.5-6 -> joakim:CAP-HORIZ
- R1, R2, R3: device resistor:R-EU_0207/7 -> resistor:R-EU_0204/5
- U$1: value BUZZER_J -> BUZZER_JL; device joakim:BUZZER_J -> joakim:BUZZER_JL
- U$2: value NFC_MODULE_V3_I2C -> NFC_MODULE_V3_I2CC; device joakim:NFC_MODULE_V3_I2C -> joakim:NFC_MODULE_V3_I2CC
Connections:
- net LED renamed LED1
- new net LED2: R4.1
- new net N$8: LED2.A, R4.2
- net GND: now also LED2.C, U$5.2; no longer S1.P1
- net SWITCH: now also U$5.1; no longer S1.S
Changed lines of the file:
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@@
 </classes>
 <parts>
-<part name="U$1" library="joakim" deviceset="BUZZER_J" device=""/>
-<part name="U$2" library="joakim" deviceset="NFC_MODULE_V3_I2C" device=""/>
+<part name="U$1" library="joakim" deviceset="BUZZER_J" device="L" value="BUZZER_JL"/>
+<part name="U$2" library="joakim" deviceset="NFC_MODULE_V3_I2C" device="C" value="NFC_MODULE_V3_I2CC"/>
 <part name="T1" library="transistor-neu-to92" deviceset="*-NPN-" device="TO92-EBC" technology="2N3904"/>
-<part name="R1" library="resistor" deviceset="R-EU_" device="0207/7" value="100"/>
-<part name="R2" library="resistor" deviceset="R-EU_" device="0207/7" value="1k"/>
-<part name="R3" library="resistor" deviceset="R-EU_" device="0207/7" value="220"/>
-<part name="C1" library="resistor" deviceset="CPOL-EU" device="E2.5-6" value="470uF"/>
+<part name="R1" library="resistor" deviceset="R-EU_" device="0204/5" value="100"/>
+<part name="R2" library="resistor" deviceset="R-EU_" device="0204/5" value="1k"/>
+<part name="R3" library="resistor" deviceset="R-EU_" device="0204/5" value="220"/>
+<part name="C1" library="joakim" deviceset="CAP-HORIZ" device="" value="470uF"/>
 <part name="GND1" library="supply1" deviceset="GND" device=""/>
 <part name="D1" library="joakim" deviceset="1N4148" device="DOJ35-5"/>
@@
 <part name="GND7" library="supply1" deviceset="GND" device=""/>
 <part name="CHARGE" library="joakim" deviceset="ST613-JACK" device=""/>
-<part name="S1" library="switch-omron" deviceset="10-XX" device=""/>
 <part name="GND8" library="supply1" deviceset="GND" device=""/>
 <part name="U$6" library="joakim" deviceset="SK12D07-SLIDE-SWITCH" device=""/>
+<part name="U$5" library="joakim" deviceset="PUSHBUTTON_2P" device=""/>
+<part name="R4" library="resistor" deviceset="R-EU_" device="0204/5" value="220"/>
+<part name="LED2" library="led" deviceset="LED" device="3MM"/>
+<part name="GND9" library="supply1" deviceset="GND" device=""/>
 </parts>
 <sheets>
@@
 </instance>
 <instance part="R3" gate="G$1" x="60.96" y="25.4"/>
-<instance part="C1" gate="G$1" x="25.4" y="33.02"/>
+<instance part="C1" gate="G$1" x="25.4" y="30.48"/>
 <instance part="GND1" gate="1" x="71.12" y="35.56"/>
 <instance part="D1" gate="G$1" x="68.58" y="53.34" smashed="yes" rot="R90">
@@
 <attribute name="NAME" x="-43.18" y="41.91" size="1.778" layer="95"/>
 </instance>
-<instance part="S1" gate="1" x="27.94" y="81.28" rot="MR270"/>
-<instance part="GND8" gate="1" x="33.02" y="76.2"/>
+<instance part="GND8" gate="1" x="38.1" y="78.74"/>
 <instance part="U$6" gate="G$1" x="-10.16" y="38.1"/>
+<instance part="U$5" gate="G$1" x="30.48" y="81.28"/>
+<instance part="R4" gate="G$1" x="60.96" y="12.7"/>
+<instance part="LED2" gate="G$1" x="68.58" y="12.7" rot="R90"/>
+<instance part="GND9" gate="1" x="76.2" y="7.62"/>
 </instances>
 <busses>
@@
 </segment>
 <segment>
-<pinref part="S1" gate="1" pin="P1"/>
+<pinref part="U$5" gate="G$1" pin="2"/>
 <pinref part="GND8" gate="1" pin="GND"/>
+</segment>
+<segment>
+<pinref part="LED2" gate="G$1" pin="C"/>
+<wire x1="73.66" y1="12.7" x2="76.2" y2="12.7" width="0.1524" layer="91"/>
+<pinref part="GND9" gate="1" pin="GND"/>
+<wire x1="76.2" y1="12.7" x2="76.2" y2="10.16" width="0.1524" layer="91"/>
 </segment>
 </net>
@@
 </segment>
 </net>
-<net name="LED" class="0">
+<net name="LED1" class="0">
 <segment>
 <pinref part="R3" gate="G$1" pin="1"/>
@@
 <wire x1="17.78" y1="101.6" x2="35.56" y2="101.6" width="0.1524" layer="91"/>
 <label x="22.86" y="101.6" size="1.778" layer="95"/>
-<pinref part="S1" gate="1" pin="S"/>
 <wire x1="22.86" y1="81.28" x2="20.32" y2="81.28" width="0.1524" layer="91"/>
 <wire x1="20.32" y1="81.28" x2="20.32" y2="93.98" width="0.1524" layer="91"/>
 <wire x1="20.32" y1="93.98" x2="35.56" y2="93.98" width="0.1524" layer="91"/>
 <wire x1="35.56" y1="93.98" x2="35.56" y2="101.6" width="0.1524" layer="91"/>
+<pinref part="U$5" gate="G$1" pin="1"/>
 </segment>
 </net>
@@
 </segment>
 </net>
+<net name="N$8" class="0">
+<segment>
+<pinref part="R4" gate="G$1" pin="2"/>
+<pinref part="LED2" gate="G$1" pin="A"/>
+</segment>
+</net>
+<net name="LED2" class="0">
+<segment>
+<pinref part="R4" gate="G$1" pin="1"/>
+<wire x1="55.88" y1="12.7" x2="40.64" y2="12.7" width="0.1524" layer="91"/>
+<label x="40.64" y="12.7" size="1.778" layer="95"/>
+</segment>
+</net>

Commit message: Hopefully final layout, tracing left
Parts:
- BATTERY_GND, BATTERY_VCC: value (none) -> DUPONT-PIN-90DEG; device joakim:MA01-1JC -> joakim:DUPONT-PIN-90DEG
- R1: value 100 -> 68
- U$2: value NFC_MODULE_V3_I2CC -> NFC_MODULE_V3_SPI; device joakim:NFC_MODULE_V3_I2CC -> joakim:NFC_MODULE_V3_SPI
- U$5: value PUSHBUTTON_2P -> PUSHBUTTON_2P6MM; device joakim:PUSHBUTTON_2P -> joakim:PUSHBUTTON_2P6MM
Connections:
- removed net IRQ: U$2.IRQ, U$4.D7
- removed net RSTO: U$2.RSTO, U$4.D8
- new net MISO: U$2.MISO, U$4.D12
- new net MOSI: U$2.MOSI, U$4.D11
- new net SCK: U$2.SCK, U$4.D13
- new net SS: U$2.SS, U$4.D10
- net BUZZER: now also U$4.D3; no longer U$4.D6
- net LED2: now also U$4.D2
- net SCL: no longer U$2.SCL
- net SDA: no longer U$2.SDA
- net SWITCH: now also U$4.D8; no longer U$4.D5
Other:
- moved on the sheet: BATTERY_GND, BATTERY_VCC
Changed lines of the file:
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@@
 <parts>
 <part name="U$1" library="joakim" deviceset="BUZZER_J" device="L" value="BUZZER_JL"/>
-<part name="U$2" library="joakim" deviceset="NFC_MODULE_V3_I2C" device="C" value="NFC_MODULE_V3_I2CC"/>
 <part name="T1" library="transistor-neu-to92" deviceset="*-NPN-" device="TO92-EBC" technology="2N3904"/>
-<part name="R1" library="resistor" deviceset="R-EU_" device="0204/5" value="100"/>
+<part name="R1" library="resistor" deviceset="R-EU_" device="0204/5" value="68"/>
 <part name="R2" library="resistor" deviceset="R-EU_" device="0204/5" value="1k"/>
 <part name="R3" library="resistor" deviceset="R-EU_" device="0204/5" value="220"/>
@@
 <part name="+3V3" library="supply1" deviceset="+3V3" device=""/>
 <part name="GND6" library="supply1" deviceset="GND" device=""/>
-<part name="BATTERY_VCC" library="joakim" deviceset="MA01-1J" device="C"/>
-<part name="BATTERY_GND" library="joakim" deviceset="MA01-1J" device="C"/>
+<part name="BATTERY_VCC" library="joakim" deviceset="DUPONT-PIN-90DEG" device=""/>
+<part name="BATTERY_GND" library="joakim" deviceset="DUPONT-PIN-90DEG" device=""/>
 <part name="+3V4" library="supply1" deviceset="+3V3" device=""/>
 <part name="GND7" library="supply1" deviceset="GND" device=""/>
@@
 <part name="GND8" library="supply1" deviceset="GND" device=""/>
 <part name="U$6" library="joakim" deviceset="SK12D07-SLIDE-SWITCH" device=""/>
-<part name="U$5" library="joakim" deviceset="PUSHBUTTON_2P" device=""/>
+<part name="U$5" library="joakim" deviceset="PUSHBUTTON_2P" device="6MM"/>
 <part name="R4" library="resistor" deviceset="R-EU_" device="0204/5" value="220"/>
 <part name="LED2" library="led" deviceset="LED" device="3MM"/>
 <part name="GND9" library="supply1" deviceset="GND" device=""/>
+<part name="U$2" library="joakim" deviceset="NFC_MODULE_V3_SPI" device=""/>
 </parts>
 <sheets>
@@
 <attribute name="NAME" x="82.55" y="58.42" size="1.778" layer="95" rot="R270"/>
 </instance>
-<instance part="U$2" gate="G$1" x="68.58" y="86.36"/>
 <instance part="T1" gate="G$1" x="68.58" y="43.18" smashed="yes">
 <attribute name="NAME" x="58.42" y="50.8" size="1.778" layer="95"/>
@@
 <instance part="LED2" gate="G$1" x="68.58" y="12.7" rot="R90"/>
 <instance part="GND9" gate="1" x="76.2" y="7.62"/>
+<instance part="U$2" gate="G$1" x="73.66" y="86.36"/>
 </instances>
 <busses>
@@
 </segment>
 <segment>
-<wire x1="-27.94" y1="50.8" x2="-25.4" y2="50.8" width="0.1524" layer="91"/>
+<wire x1="-30.48" y1="50.8" x2="-25.4" y2="50.8" width="0.1524" layer="91"/>
 <wire x1="-25.4" y1="50.8" x2="-20.32" y2="50.8" width="0.1524" layer="91"/>
 <wire x1="-20.32" y1="50.8" x2="-20.32" y2="48.26" width="0.1524" layer="91"/>
@@
 </segment>
 <segment>
-<pinref part="U$2" gate="G$1" pin="GND"/>
-<wire x1="58.42" y1="93.98" x2="55.88" y2="93.98" width="0.1524" layer="91"/>
+<wire x1="63.5" y1="93.98" x2="55.88" y2="93.98" width="0.1524" layer="91"/>
 <wire x1="55.88" y1="93.98" x2="55.88" y2="99.06" width="0.1524" layer="91"/>
 <pinref part="GND6" gate="1" pin="GND"/>
 <wire x1="55.88" y1="99.06" x2="53.34" y2="99.06" width="0.1524" layer="91"/>
+<pinref part="U$2" gate="G$1" pin="GND"/>
 </segment>
 <segment>
@@
 <pinref part="+3V3" gate="G$1" pin="+3V3"/>
 <wire x1="45.72" y1="93.98" x2="45.72" y2="91.44" width="0.1524" layer="91"/>
+<wire x1="45.72" y1="91.44" x2="63.5" y2="91.44" width="0.1524" layer="91"/>
 <pinref part="U$2" gate="G$1" pin="VCC"/>
-<wire x1="45.72" y1="91.44" x2="58.42" y2="91.44" width="0.1524" layer="91"/>
 </segment>
 <segment>
@@
 </segment>
 <segment>
-<pinref part="U$4" gate="G$1" pin="D6"/>
-<wire x1="17.78" y1="104.14" x2="33.02" y2="104.14" width="0.1524" layer="91"/>
-<label x="22.86" y="104.14" size="1.778" layer="95"/>
+<pinref part="U$4" gate="G$1" pin="D3"/>
+<wire x1="17.78" y1="96.52" x2="33.02" y2="96.52" width="0.1524" layer="91"/>
+<label x="22.86" y="96.52" size="1.778" layer="95"/>
 </segment>
 </net>
@@
 <label x="-30.48" y="78.74" size="1.778" layer="95"/>
 </segment>
-<segment>
-<pinref part="U$2" gate="G$1" pin="SDA"/>
-<wire x1="58.42" y1="88.9" x2="45.72" y2="88.9" width="0.1524" layer="91"/>
-<label x="45.72" y="88.9" size="1.778" layer="95"/>
-</segment>
 </net>
 <net name="SCL" class="0">
@@
 <wire x1="-20.32" y1="76.2" x2="-30.48" y2="76.2" width="0.1524" layer="91"/>
 <label x="-30.48" y="76.2" size="1.778" layer="95"/>
-</segment>
-<segment>
-<pinref part="U$2" gate="G$1" pin="SCL"/>
-<wire x1="58.42" y1="86.36" x2="45.72" y2="86.36" width="0.1524" layer="91"/>
-<label x="45.72" y="86.36" size="1.778" layer="95"/>
-</segment>
-</net>
-<net name="IRQ" class="0">
-<segment>
-<pinref part="U$2" gate="G$1" pin="IRQ"/>
-<wire x1="58.42" y1="83.82" x2="45.72" y2="83.82" width="0.1524" layer="91"/>
-<label x="45.72" y="83.82" size="1.778" layer="95"/>
-</segment>
-<segment>
-<pinref part="U$4" gate="G$1" pin="D7"/>
-<wire x1="17.78" y1="106.68" x2="33.02" y2="106.68" width="0.1524" layer="91"/>
-<label x="22.86" y="106.68" size="1.778" layer="95"/>
-</segment>
-</net>
-<net name="RSTO" class="0">
-<segment>
-<pinref part="U$2" gate="G$1" pin="RSTO"/>
-<wire x1="58.42" y1="81.28" x2="45.72" y2="81.28" width="0.1524" layer="91"/>
-<label x="45.72" y="81.28" size="1.778" layer="95"/>
-</segment>
-<segment>
-<pinref part="U$4" gate="G$1" pin="D8"/>
-<wire x1="17.78" y1="109.22" x2="33.02" y2="109.22" width="0.1524" layer="91"/>
-<label x="22.86" y="109.22" size="1.778" layer="95"/>
 </segment>
 </net>
@@
 <wire x1="-25.4" y1="35.56" x2="-25.4" y2="22.86" width="0.1524" layer="91"/>
 <pinref part="BATTERY_VCC" gate="G$1" pin="1"/>
-<wire x1="-25.4" y1="22.86" x2="-27.94" y2="22.86" width="0.1524" layer="91"/>
+<wire x1="-25.4" y1="22.86" x2="-30.48" y2="22.86" width="0.1524" layer="91"/>
 </segment>
 </net>
 <net name="SWITCH" class="0">
 <segment>
-<pinref part="U$4" gate="G$1" pin="D5"/>
-<wire x1="17.78" y1="101.6" x2="35.56" y2="101.6" width="0.1524" layer="91"/>
-<label x="22.86" y="101.6" size="1.778" layer="95"/>
 <wire x1="22.86" y1="81.28" x2="20.32" y2="81.28" width="0.1524" layer="91"/>
-<wire x1="20.32" y1="81.28" x2="20.32" y2="93.98" width="0.1524" layer="91"/>
-<wire x1="20.32" y1="93.98" x2="35.56" y2="93.98" width="0.1524" layer="91"/>
-<wire x1="35.56" y1="93.98" x2="35.56" y2="101.6" width="0.1524" layer="91"/>
+<wire x1="20.32" y1="81.28" x2="20.32" y2="88.9" width="0.1524" layer="91"/>
+<wire x1="20.32" y1="88.9" x2="35.56" y2="88.9" width="0.1524" layer="91"/>
+<wire x1="35.56" y1="88.9" x2="35.56" y2="109.22" width="0.1524" layer="91"/>
 <pinref part="U$5" gate="G$1" pin="1"/>
+<pinref part="U$4" gate="G$1" pin="D8"/>
+<wire x1="35.56" y1="109.22" x2="17.78" y2="109.22" width="0.1524" layer="91"/>
+<label x="22.86" y="109.22" size="1.778" layer="95"/>
 </segment>
 </net>
@@
 <label x="40.64" y="12.7" size="1.778" layer="95"/>
 </segment>
-</net>
+<segment>
+<pinref part="U$4" gate="G$1" pin="D2"/>
+<wire x1="17.78" y1="93.98" x2="33.02" y2="93.98" width="0.1524" layer="91"/>
+<label x="22.86" y="93.98" size="1.778" layer="95"/>
+</segment>
+</net>
+<net name="SCK" class="0">
+<segment>
+<wire x1="63.5" y1="88.9" x2="45.72" y2="88.9" width="0.1524" layer="91"/>
+<label x="45.72" y="88.9" size="1.778" layer="95"/>
+<pinref part="U$2" gate="G$1" pin="SCK"/>
+</segment>
+<segment>
+<pinref part="U$4" gate="G$1" pin="D13"/>
+<wire x1="-20.32" y1="104.14" x2="-35.56" y2="104.14" width="0.1524" layer="91"/>
+<label x="-35.56" y="104.14" size="1.778" layer="95"/>
+</segment>
+</net>
+<net name="MISO" class="0">
+<segment>
+<wire x1="63.5" y1="86.36" x2="45.72" y2="86.36" width="0.1524" layer="91"/>
+<label x="45.72" y="86.36" size="1.778" layer="95"/>
+<pinref part="U$2" gate="G$1" pin="MISO"/>
+</segment>
+<segment>
+<pinref part="U$4" gate="G$1" pin="D12"/>
+<wire x1="-20.32" y1="106.68" x2="-35.56" y2="106.68" width="0.1524" layer="91"/>
+<label x="-35.56" y="106.68" size="1.778" layer="95"/>
+</segment>
+</net>
+<net name="MOSI" class="0">
+<segment>
+<wire x1="63.5" y1="83.82" x2="45.72" y2="83.82" width="0.1524" layer="91"/>
+<label x="45.72" y="83.82" size="1.778" layer="95"/>
+<pinref part="U$2" gate="G$1" pin="MOSI"/>
+</segment>
+<segment>
+<pinref part="U$4" gate="G$1" pin="D11"/>
+<wire x1="-20.32" y1="109.22" x2="-35.56" y2="109.22" width="0.1524" layer="91"/>
+<label x="-35.56" y="109.22" size="1.778" layer="95"/>
+</segment>
+</net>
+<net name="SS" class="0">
+<segment>
+<wire x1="63.5" y1="81.28" x2="45.72" y2="81.28" width="0.1524" layer="91"/>
+<label x="45.72" y="81.28" size="1.778" layer="95"/>
+<pinref part="U$2" gate="G$1" pin="SS"/>
+</segment>
+<segment>
+<pinref part="U$4" gate="G$1" pin="D10"/>
+<wire x1="-20.32" y1="111.76" x2="-35.56" y2="111.76" width="0.1524" layer="91"/>
+<label x="-35.56" y="111.76" size="1.778" layer="95"/>
+</segment>
+</net>

Commit message: Traced and fixed most silk screening
Parts:
- added SV1, SV2: (no value), joakim:MA01-1JC
- LED1, LED2: device led:LED3MM -> joakim:LED_J3MM-LEFT
- U$2: value NFC_MODULE_V3_SPI -> NFC_MODULE_V3_SPINH; device joakim:NFC_MODULE_V3_SPI -> joakim:NFC_MODULE_V3_SPINH
Connections:
- net GND: now also SV1.1
- net N$6: now also SV2.1
Other:
- moved on the sheet: BATTERY_GND, BATTERY_VCC
Changed lines of the file:
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@@
 <part name="D1" library="joakim" deviceset="1N4148" device="DOJ35-5"/>
 <part name="+3V1" library="supply1" deviceset="+3V3" device=""/>
-<part name="LED1" library="led" deviceset="LED" device="3MM"/>
+<part name="LED1" library="joakim" deviceset="LED_J" device="3MM-LEFT"/>
 <part name="GND2" library="supply1" deviceset="GND" device=""/>
 <part name="U$3" library="joakim" deviceset="VOLT_BOOST" device=""/>
@@
 <part name="U$5" library="joakim" deviceset="PUSHBUTTON_2P" device="6MM"/>
 <part name="R4" library="resistor" deviceset="R-EU_" device="0204/5" value="220"/>
-<part name="LED2" library="led" deviceset="LED" device="3MM"/>
+<part name="LED2" library="joakim" deviceset="LED_J" device="3MM-LEFT"/>
 <part name="GND9" library="supply1" deviceset="GND" device=""/>
-<part name="U$2" library="joakim" deviceset="NFC_MODULE_V3_SPI" device=""/>
+<part name="U$2" library="joakim" deviceset="NFC_MODULE_V3_SPI" device="NH" value="NFC_MODULE_V3_SPINH"/>
+<part name="SV1" library="joakim" deviceset="MA01-1J" device="C"/>
+<part name="SV2" library="joakim" deviceset="MA01-1J" device="C"/>
 </parts>
 <sheets>
@@
 <attribute name="VALUE" x="33.02" y="43.18" size="1.778" layer="96" rot="R180"/>
 </instance>
-<instance part="GND5" gate="1" x="-20.32" y="45.72"/>
+<instance part="GND5" gate="1" x="-15.24" y="53.34"/>
 <instance part="U$4" gate="G$1" x="0" y="93.98" rot="R180"/>
 <instance part="+3V3" gate="G$1" x="45.72" y="96.52"/>
 <instance part="GND6" gate="1" x="53.34" y="96.52"/>
-<instance part="BATTERY_VCC" gate="G$1" x="-35.56" y="22.86" smashed="yes">
-<attribute name="VALUE" x="-36.83" y="17.78" size="1.778" layer="96"/>
-<attribute name="NAME" x="-36.83" y="16.002" size="1.778" layer="95"/>
-</instance>
-<instance part="BATTERY_GND" gate="G$1" x="-35.56" y="50.8" smashed="yes">
-<attribute name="VALUE" x="-36.83" y="45.72" size="1.778" layer="96"/>
-<attribute name="NAME" x="-36.83" y="54.102" size="1.778" layer="95"/>
+<instance part="BATTERY_VCC" gate="G$1" x="-35.56" y="20.32" smashed="yes">
+<attribute name="VALUE" x="-49.53" y="15.24" size="1.778" layer="96"/>
+<attribute name="NAME" x="-49.53" y="10.922" size="1.778" layer="95"/>
+</instance>
+<instance part="BATTERY_GND" gate="G$1" x="-35.56" y="55.88" smashed="yes">
+<attribute name="VALUE" x="-49.53" y="60.96" size="1.778" layer="96"/>
+<attribute name="NAME" x="-49.53" y="64.262" size="1.778" layer="95"/>
 </instance>
 <instance part="+3V4" gate="G$1" x="-35.56" y="93.98"/>
@@
 <instance part="GND9" gate="1" x="76.2" y="7.62"/>
 <instance part="U$2" gate="G$1" x="73.66" y="86.36"/>
+<instance part="SV1" gate="G$1" x="-38.1" y="50.8" smashed="yes">
+<attribute name="VALUE" x="-39.37" y="45.72" size="1.778" layer="96"/>
+<attribute name="NAME" x="-31.75" y="46.482" size="1.778" layer="95"/>
+</instance>
+<instance part="SV2" gate="G$1" x="-38.1" y="25.4"/>
 </instances>
 <busses>
@@
 </segment>
 <segment>
-<wire x1="-30.48" y1="50.8" x2="-25.4" y2="50.8" width="0.1524" layer="91"/>
-<wire x1="-25.4" y1="50.8" x2="-20.32" y2="50.8" width="0.1524" layer="91"/>
-<wire x1="-20.32" y1="50.8" x2="-20.32" y2="48.26" width="0.1524" layer="91"/>
+<wire x1="-30.48" y1="55.88" x2="-25.4" y2="55.88" width="0.1524" layer="91"/>
+<wire x1="-25.4" y1="55.88" x2="-15.24" y2="55.88" width="0.1524" layer="91"/>
 <pinref part="GND5" gate="1" pin="GND"/>
 <pinref part="BATTERY_GND" gate="G$1" pin="1"/>
@@
 <wire x1="-30.48" y1="40.64" x2="-25.4" y2="40.64" width="0.1524" layer="91"/>
 <wire x1="-25.4" y1="40.64" x2="-25.4" y2="50.8" width="0.1524" layer="91"/>
+<junction x="-25.4" y="55.88"/>
+<pinref part="SV1" gate="G$1" pin="1"/>
+<wire x1="-25.4" y1="50.8" x2="-25.4" y2="55.88" width="0.1524" layer="91"/>
+<wire x1="-30.48" y1="50.8" x2="-25.4" y2="50.8" width="0.1524" layer="91"/>
 <junction x="-25.4" y="50.8"/>
 </segment>
@@
 <pinref part="CHARGE" gate="G$1" pin="3"/>
 <wire x1="-30.48" y1="35.56" x2="-25.4" y2="35.56" width="0.1524" layer="91"/>
-<wire x1="-25.4" y1="35.56" x2="-25.4" y2="22.86" width="0.1524" layer="91"/>
+<wire x1="-25.4" y1="35.56" x2="-25.4" y2="25.4" width="0.1524" layer="91"/>
 <pinref part="BATTERY_VCC" gate="G$1" pin="1"/>
-<wire x1="-25.4" y1="22.86" x2="-30.48" y2="22.86" width="0.1524" layer="91"/>
-</segment>
-</net>
+<wire x1="-25.4" y1="25.4" x2="-25.4" y2="20.32" width="0.1524" layer="91"/>
+<wire x1="-25.4" y1="20.32" x2="-30.48" y2="20.32" width="0.1524" layer="91"/>
+<pinref part="SV2" gate="G$1" pin="1"/>
+<wire x1="-30.48" y1="25.4" x2="-25.4" y2="25.4" width="0.1524" layer="91"/>
+<junction x="-25.4" y="25.4"/>
+</segment>
+</net>
